File: kicad/emuecu_2.kicad_pcb (KiCad board)
At the start: 2 copper layers, 97 parts, among them P1 INJECTOR, P10 PUMP, P11 AIR_TEMP, P12 I2C, P13 SERIAL, P14 SPI, P2 FAN/PUMP, P3 IGNITION, P4 LOAD, P5 THROTTLE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

Commit message: updates to schematic, minor changes to map
Parts:
- removed C7: 4.7uF, C1V5
- removed L3: 47uH, C2V8
- added R34: 100, R4, F.Cu at (144.1, 69.2)
- added R35: 100, R4, F.Cu at (144.1, 79.4)
- P11: value AIR_TEMP -> AIR TEMP; footprint SIL-3 -> SIL-2
- P8: value ENGINE_TEMP -> ENG TEMP; footprint SIL-3 -> SIL-2
- R12, R21: value 20k -> 100k
- R5: value 470 -> 200
- Z2: value IN4732 (4.7V) -> IN5919BG (5.6V)
- moved C6 35.5 mm to (160.0, 48.3), turned to 180 degrees
- moved Z1 9.00 mm to (207.4, 43.2)
- moved D1 6.99 mm to (186.7, 44.5)
- moved T4 6.99 mm to (193.7, 44.5)
- moved D3 5.97 mm to (200.4, 44.5)
- moved R2 3.61 mm to (204.7, 44.2)
- moved P13 3.17 mm to (134.0, 54.6)
- moved R27 3.17 mm to (141.6, 52.1)
- moved R28 3.17 mm to (156.8, 52.1)
- moved R29 3.17 mm to (141.6, 54.6)
- moved R30 3.17 mm to (156.8, 54.6)
- moved Z8 3.17 mm to (156.8, 57.1)
- moved Z9 3.17 mm to (141.6, 57.1)
- moved R4 2.62 mm to (208.3, 62.2)
- moved D12 2.54 mm to (142.9, 87.0)
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Connections:
- C6 pad 1: N-000005 (its old number) -> +12V
- L1 pad 2: N-000005 (its old number) -> +12V
- P11 pad 1: N-0000069 (its old number) -> +5C
- P11 pad 2: +5C -> N-0000011
- P6 pad 2: +5C -> N-0000027
- P7 pad 2: +5C -> N-0000064
- P8 pad 1: N-0000067 (its old number) -> +5C
- P8 pad 2: +5C -> N-0000014
- R12 pad 1: +5C -> N-0000014
- R12 pad 2: N-0000067 (its old number) -> SGND
- R13 pad 1: N-0000067 (its old number) -> N-0000014
- R21 pad 1: +5C -> N-0000011
- R21 pad 2: N-0000069 (its old number) -> SGND
- R22 pad 1: N-0000069 (its old number) -> N-0000011
- U1 pad 30: N-000005 (its old number) -> +12V
Routing:
- net +12V: track 0.00 -> 104.1 mm, vias 0 -> 1
- net GND: track 131.9 -> 203.1 mm
- net N-000005 (its old number): track 50.1 -> 0.00 mm
- net N-000005: track 95.1 -> 45.9 mm, vias 0 -> 1
- net +5V: track 53.3 -> 100.2 mm, vias 1 -> 2
- net +5C: track 190.8 -> 148.6 mm
- net N-000006: track 0.00 -> 41.0 mm
- net N-0000066: track 61.4 -> 98.3 mm
- net N-0000024: track 0.00 -> 32.0 mm
- net N-0000067: track 58.2 -> 85.6 mm
- net N-0000043: track 40.6 -> 67.7 mm, vias 0 -> 1
- net N-0000065: track 0.00 -> 14.6 mm, vias 0 -> 1
- net N-0000069 (its old number): track 13.8 -> 0.00 mm
- net N-0000067 (its old number): track 13.8 -> 0.00 mm
- net SGND: track 2.54 -> 15.3 mm
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- added copper zone on F.Cu, net GND
- added copper zone on F.Cu, net SGND

Commit message: update to kicad 5.1
Parts:
- L1, L2: footprint C2V8 -> Inductor_THT:L_Radial_D8.7mm_P5.00mm_Fastron_07HCP
- P12: footprint SIL-4 -> Connector_PinHeader_2.54mm:PinHeader_1x04_P2.54mm_Vertical
- P13: value SERIAL -> Serial
- R12, R21: value 100k -> 22k
- U1: footprint arduino_nano -> arduino:arduino_nano
- moved P12 3.81 mm to (188.6, 66.7), turned to 0 degrees
- moved L1 2.54 mm to (164.5, 45.1), turned to 90 degrees
- moved L2 2.54 mm to (157.5, 42.5)
Connections:
- D2 pad 1: N-0000020 -> Net-(D2-Pad1)
- L1 pad 1: N-0000020 -> +12V
- L1 pad 2: +12V -> Net-(D2-Pad1)
- U1 pad 10: (no net) -> Net-(U1-Pad10)
- U1 pad 17: (no net) -> Net-(U1-Pad17)
- U1 pad 18: (no net) -> Net-(U1-Pad18)
- U1 pad 21: (no net) -> Net-(U1-Pad21)
- U1 pad 22: (no net) -> Net-(U1-Pad22)
- U1 pad 25: (no net) -> Net-(U1-Pad25)
- U1 pad 26: (no net) -> Net-(U1-Pad26)
- U1 pad 28: (no net) -> Net-(U1-Pad28)
- U1 pad 3: (no net) -> Net-(U1-Pad3)
- U5 pad 1: (no net) -> Net-(U5-Pad1)
- U5 pad 4: (no net) -> Net-(U5-Pad4)
- U5 pad 7: (no net) -> Net-(U5-Pad7)
Routing:
- net Net-(D2-Pad1): track 0.00 -> 15.5 mm
- net N-0000020: track 15.5 -> 0.00 mm
